Commit message: feat: hiwonderbot with custom gripper urdf and debug print for link and limits in  test_urdf

File: assets/Hiwonder_description/urdf/Hiwonder.xacro (robot description, xacro)
@@ -26,5 +26,5 @@
 <link name="second_link_1">
   <inertial>
-    <origin xyz="0.001515564224594493 1.7928644227976909e-06 0.024809430057853542" rpy="0 0 0"/>
+    <origin xyz="0.001515476232598548 -1.6684843491224233e-05 0.02480943005786166" rpy="0 0 0"/>
     <mass value="0.37909012139587217"/>
     <inertia ixx="0.000161" iyy="0.00016" izz="0.000201" ixy="0.0" iyz="0.0" ixz="-6e-06"/>
@@ -46,10 +46,10 @@
 <link name="third_link_1">
   <inertial>
-    <origin xyz="-0.027698296621640646 0.03104027583896596 0.04168837472454898" rpy="0 0 0"/>
+    <origin xyz="-0.027343180150573892 0.029293876913652088 0.04316047625280414" rpy="0 0 0"/>
     <mass value="0.16226233466168985"/>
-    <inertia ixx="0.000203" iyy="0.000223" izz="0.000169" ixy="-0.0" iyz="-9e-05" ixz="-0.0"/>
-  </inertial>
-  <visual>
-    <origin xyz="-0.028042 -0.046304 -0.095801" rpy="0 0 0"/>
+    <inertia ixx="0.000203" iyy="0.000231" izz="0.00016" ixy="0.0" iyz="-8.7e-05" ixz="-1e-06"/>
+  </inertial>
+  <visual>
+    <origin xyz="-0.027918 -0.045963 -0.095801" rpy="0 0 0"/>
     <geometry>
       <mesh filename="package://Hiwonder_description/meshes/third_link_1.stl" scale="0.001 0.001 0.001"/>
@@ -58,5 +58,5 @@
   </visual>
   <collision>
-    <origin xyz="-0.028042 -0.046304 -0.095801" rpy="0 0 0"/>
+    <origin xyz="-0.027918 -0.045963 -0.095801" rpy="0 0 0"/>
     <geometry>
       <mesh filename="package://Hiwonder_description/meshes/third_link_1.stl" scale="0.001 0.001 0.001"/>
@@ -66,10 +66,10 @@
 <link name="fourth_link_1">
   <inertial>
-    <origin xyz="-0.025726869907649247 -0.014316329119973825 0.01864921442376344" rpy="0 0 0"/>
+    <origin xyz="-0.025886175644017836 -0.012863720404565696 0.019469646301894933" rpy="0 0 0"/>
     <mass value="0.2923899366437736"/>
-    <inertia ixx="0.000208" iyy="0.000198" izz="0.000149" ixy="1e-06" iyz="8.9e-05" ixz="-2e-06"/>
-  </inertial>
-  <visual>
-    <origin xyz="-0.028042 -0.108414 -0.179217" rpy="0 0 0"/>
+    <inertia ixx="0.000208" iyy="0.000208" izz="0.000139" ixy="1e-06" iyz="8.6e-05" ixz="-1e-06"/>
+  </inertial>
+  <visual>
+    <origin xyz="-0.028625 -0.103903 -0.182163" rpy="0 0 0"/>
     <geometry>
       <mesh filename="package://Hiwonder_description/meshes/fourth_link_1.stl" scale="0.001 0.001 0.001"/>
@@ -78,5 +78,5 @@
   </visual>
   <collision>
-    <origin xyz="-0.028042 -0.108414 -0.179217" rpy="0 0 0"/>
+    <origin xyz="-0.028625 -0.103903 -0.182163" rpy="0 0 0"/>
     <geometry>
       <mesh filename="package://Hiwonder_description/meshes/fourth_link_1.stl" scale="0.001 0.001 0.001"/>
@@ -86,10 +86,10 @@
 <link name="fifth_link_1">
   <inertial>
-    <origin xyz="0.024821511351616442 -0.02017792012395629 -0.009479484341226002" rpy="0 0 0"/>
+    <origin xyz="0.024573606883266846 -0.020492170669535084 -0.009450750798881968" rpy="0 0 0"/>
     <mass value="0.29380221652800204"/>
-    <inertia ixx="0.000201" iyy="0.000102" izz="0.000168" ixy="-6e-06" iyz="3e-06" ixz="-1e-06"/>
-  </inertial>
-  <visual>
-    <origin xyz="0.0285 -0.054537 -0.249542" rpy="0 0 0"/>
+    <inertia ixx="0.000201" iyy="0.000102" izz="0.000168" ixy="-8e-06" iyz="3e-06" ixz="-1e-06"/>
+  </inertial>
+  <visual>
+    <origin xyz="0.028518 -0.05501 -0.255576" rpy="0 0 0"/>
     <geometry>
       <mesh filename="package://Hiwonder_description/meshes/fifth_link_1.stl" scale="0.001 0.001 0.001"/>
@@ -98,5 +98,5 @@
   </visual>
   <collision>
-    <origin xyz="0.0285 -0.054537 -0.249542" rpy="0 0 0"/>
+    <origin xyz="0.028518 -0.05501 -0.255576" rpy="0 0 0"/>
     <geometry>
       <mesh filename="package://Hiwonder_description/meshes/fifth_link_1.stl" scale="0.001 0.001 0.001"/>
@@ -106,10 +106,10 @@
 <link name="sixth_link_1">
   <inertial>
-    <origin xyz="-0.010116017933357755 -0.02248782358725894 -0.010025570313181048" rpy="0 0 0"/>
-    <mass value="0.1573394430491276"/>
-    <inertia ixx="4.4e-05" iyy="6.2e-05" izz="4.9e-05" ixy="-3e-06" iyz="-3e-06" ixz="-0.0"/>
-  </inertial>
-  <visual>
-    <origin xyz="0.003224 0.009777 -0.249338" rpy="0 0 0"/>
+    <origin xyz="-0.00040907580167635384 -0.046363022962390074 -0.0038289785318220693" rpy="0 0 0"/>
+    <mass value="0.5747761409814244"/>
+    <inertia ixx="0.000539" iyy="0.000272" izz="0.000341" ixy="-3e-06" iyz="-5.3e-05" ixz="0.0"/>
+  </inertial>
+  <visual>
+    <origin xyz="0.004028 0.009607 -0.255463" rpy="0 0 0"/>
     <geometry>
       <mesh filename="package://Hiwonder_description/meshes/sixth_link_1.stl" scale="0.001 0.001 0.001"/>
@@ -118,5 +118,5 @@
   </visual>
   <collision>
-    <origin xyz="0.003224 0.009777 -0.249338" rpy="0 0 0"/>
+    <origin xyz="0.004028 0.009607 -0.255463" rpy="0 0 0"/>
     <geometry>
       <mesh filename="package://Hiwonder_description/meshes/sixth_link_1.stl" scale="0.001 0.001 0.001"/>
@@ -124,58 +124,118 @@
   </collision>
 </link>
-<link name="seventh_link_1">
-  <inertial>
-    <origin xyz="-0.0013419611646981527 -0.04606682458154797 -3.0105183902451316e-05" rpy="0 0 0"/>
-    <mass value="0.11741284268359674"/>
-    <inertia ixx="8.6e-05" iyy="5.6e-05" izz="0.000112" ixy="0.0" iyz="-4e-06" ixz="2.3e-05"/>
-  </inertial>
-  <visual>
-    <origin xyz="0.002147 0.017264 -0.250874" rpy="0 0 0"/>
-    <geometry>
-      <mesh filename="package://Hiwonder_description/meshes/seventh_link_1.stl" scale="0.001 0.001 0.001"/>
-    </geometry>
-    <material name="silver"/>
-  </visual>
-  <collision>
-    <origin xyz="0.002147 0.017264 -0.250874" rpy="0 0 0"/>
-    <geometry>
-      <mesh filename="package://Hiwonder_description/meshes/seventh_link_1.stl" scale="0.001 0.001 0.001"/>
-    </geometry>
-  </collision>
-</link>
-<joint name="Revolute 13" type="continuous">
+<link name="left_finger_1">
+  <inertial>
+    <origin xyz="0.22614187622313073 -0.16382465810915833 -0.07528218342616169" rpy="0 0 0"/>
+    <mass value="0.07506411850762539"/>
+    <inertia ixx="3.9e-05" iyy="2.9e-05" izz="2e-05" ixy="-0.0" iyz="-1.2e-05" ixz="0.0"/>
+  </inertial>
+  <visual>
+    <origin xyz="0.239188 -0.06338 -0.290008" rpy="0 0 0"/>
+    <geometry>
+      <mesh filename="package://Hiwonder_description/meshes/left_finger_1.stl" scale="0.001 0.001 0.001"/>
+    </geometry>
+    <material name="silver"/>
+  </visual>
+  <collision>
+    <origin xyz="0.239188 -0.06338 -0.290008" rpy="0 0 0"/>
+    <geometry>
+      <mesh filename="package://Hiwonder_description/meshes/left_finger_1.stl" scale="0.001 0.001 0.001"/>
+    </geometry>
+  </collision>
+</link>
+<link name="right_finger_1">
+  <inertial>
+    <origin xyz="0.23353711603941524 -0.16423216885509756 0.009285417328035783" rpy="0 0 0"/>
+    <mass value="0.07962832262347441"/>
+    <inertia ixx="4e-05" iyy="3.6e-05" izz="2.7e-05" ixy="-8e-06" iyz="1.2e-05" ixz="8e-06"/>
+  </inertial>
+  <visual>
+    <origin xyz="0.239287 -0.063365 -0.267308" rpy="0 0 0"/>
+    <geometry>
+      <mesh filename="package://Hiwonder_description/meshes/right_finger_1.stl" scale="0.001 0.001 0.001"/>
+    </geometry>
+    <material name="silver"/>
+  </visual>
+  <collision>
+    <origin xyz="0.239287 -0.063365 -0.267308" rpy="0 0 0"/>
+    <geometry>
+      <mesh filename="package://Hiwonder_description/meshes/right_finger_1.stl" scale="0.001 0.001 0.001"/>
+    </geometry>
+  </collision>
+</link>
+<link name="gear_link_1">
+  <inertial>
+    <origin xyz="-6.661216082451751e-05 -0.008319512177334093 7.260586570295713e-05" rpy="0 0 0"/>
+    <mass value="0.025254124812982604"/>
+    <inertia ixx="2e-06" iyy="1e-06" izz="2e-06" ixy="-0.0" iyz="0.0" ixz="0.0"/>
+  </inertial>
+  <visual>
+    <origin xyz="0.004496 0.068042 -0.245637" rpy="0 0 0"/>
+    <geometry>
+      <mesh filename="package://Hiwonder_description/meshes/gear_link_1.stl" scale="0.001 0.001 0.001"/>
+    </geometry>
+    <material name="silver"/>
+  </visual>
+  <collision>
+    <origin xyz="0.004496 0.068042 -0.245637" rpy="0 0 0"/>
+    <geometry>
+      <mesh filename="package://Hiwonder_description/meshes/gear_link_1.stl" scale="0.001 0.001 0.001"/>
+    </geometry>
+  </collision>
+</link>
+<joint name="Revolute 13" type="revolute">
   <origin xyz="0.0 0.056304 0.060801" rpy="0 0 0"/>
   <parent link="base_link"/>
   <child link="second_link_1"/>
   <axis xyz="0.0 0.0 -1.0"/>
-</joint>
-<joint name="Revolute 14" type="continuous">
-  <origin xyz="0.028042 -0.01 0.035" rpy="0 0 0"/>
+  <limit upper="1.570796" lower="-1.570796" effort="100" velocity="100"/>
+</joint>
+<joint name="Revolute 14" type="revolute">
+  <origin xyz="0.027918 -0.010341 0.035" rpy="0 0 0"/>
   <parent link="second_link_1"/>
   <child link="third_link_1"/>
-  <axis xyz="-1.0 -0.0 0.0"/>
-</joint>
-<joint name="Revolute 15" type="continuous">
-  <origin xyz="0.0 0.06211 0.083416" rpy="0 0 0"/>
+  <axis xyz="-0.999926 0.012192 -0.0"/>
+  <limit upper="0.785398" lower="-2.094395" effort="100" velocity="100"/>
+</joint>
+<joint name="Revolute 15" type="revolute">
+  <origin xyz="0.000707 0.05794 0.086362" rpy="0 0 0"/>
   <parent link="third_link_1"/>
   <child link="fourth_link_1"/>
-  <axis xyz="-1.0 0.0 0.0"/>
-</joint>
-<joint name="Revolute 16" type="continuous">
-  <origin xyz="-0.056542 -0.053877 0.070325" rpy="0 0 0"/>
+  <axis xyz="-0.999926 0.012192 -0.0"/>
+  <limit upper="2.879793" lower="-0.261799" effort="100" velocity="100"/>
+</joint>
+<joint name="Revolute 16" type="revolute">
+  <origin xyz="-0.057143 -0.048893 0.073413" rpy="0 0 0"/>
   <parent link="fourth_link_1"/>
   <child link="fifth_link_1"/>
-  <axis xyz="1.0 0.0 -0.0"/>
-</joint>
-<joint name="Revolute 17" type="continuous">
-  <origin xyz="0.025276 -0.064314 -0.000204" rpy="0 0 0"/>
+  <axis xyz="0.999926 -0.012192 0.0"/>
+  <limit upper="0.698132" lower="-2.443461" effort="100" velocity="100"/>
+</joint>
+<joint name="Revolute 19" type="continuous">
+  <origin xyz="0.02449 -0.064617 -0.000113" rpy="0 0 0"/>
   <parent link="fifth_link_1"/>
   <child link="sixth_link_1"/>
-  <axis xyz="-0.004192 0.999965 -0.007266"/>
-</joint>
-<joint name="Rigid 18" type="fixed">
-  <origin xyz="0.001077 -0.007487 0.001536" rpy="0 0 0"/>
+  <axis xyz="0.008 0.99993 -0.008671"/>
+</joint>
+<joint name="Slider 20" type="prismatic">
+  <origin xyz="-0.23516 0.072987 0.034545" rpy="0 0 0"/>
   <parent link="sixth_link_1"/>
-  <child link="seventh_link_1"/>
+  <child link="left_finger_1"/>
+  <axis xyz="-0.004274 0.008705 0.999953"/>
+  <limit upper="0.015" lower="-0.015" effort="100" velocity="100"/>
+</joint>
+<joint name="Slider 21" type="prismatic">
+  <origin xyz="-0.235259 0.072972 0.011845" rpy="0 0 0"/>
+  <parent link="sixth_link_1"/>
+  <child link="right_finger_1"/>
+  <axis xyz="-0.004274 0.008705 0.999953"/>
+  <limit upper="0.015" lower="-0.015" effort="100" velocity="100"/>
+</joint>
+<joint name="Revolute 22" type="revolute">
+  <origin xyz="-0.000468 -0.058435 -0.009826" rpy="0 0 0"/>
+  <parent link="sixth_link_1"/>
+  <child link="gear_link_1"/>
+  <axis xyz="0.008 0.99993 -0.008671"/>
+  <limit upper="5.585054" lower="0.872665" effort="100" velocity="100"/>
 </joint>
 </robot>
