Commit message: wip: urdf related changes
previous urdf file contains bug.
new code files are also not updated accoring to the latest urdf files. this is a WIP

File: assets/Hiwonder_description/urdf/Hiwonder.xacro (robot description, xacro)
@@ -26,5 +26,5 @@
 <link name="second_link_1">
   <inertial>
-    <origin xyz="0.0015155642244600231 1.7928644227699353e-06 0.024809430057861744" rpy="0 0 0"/>
+    <origin xyz="0.0015155642244600214 1.7928644227976909e-06 0.024809430057861744" rpy="0 0 0"/>
     <mass value="0.37909012139587217"/>
     <inertia ixx="0.000161" iyy="0.00016" izz="0.000201" ixy="0.0" iyz="0.0" ixz="-6e-06"/>
@@ -44,12 +44,72 @@
   </collision>
 </link>
+<link name="sixth_link_1">
+  <inertial>
+    <origin xyz="0.00015608115480679387 0.04624085970692193 0.0051057604762696635" rpy="0 0 0"/>
+    <mass value="0.5747761409814244"/>
+    <inertia ixx="0.000539" iyy="0.000275" izz="0.000338" ixy="-1e-06" iyz="-5.5e-05" ixz="-1e-06"/>
+  </inertial>
+  <visual>
+    <origin xyz="0.004904 -0.303181 -0.097772" rpy="0 0 0"/>
+    <geometry>
+      <mesh filename="package://Hiwonder_description/meshes/sixth_link_1.stl" scale="0.001 0.001 0.001"/>
+    </geometry>
+    <material name="silver"/>
+  </visual>
+  <collision>
+    <origin xyz="0.004904 -0.303181 -0.097772" rpy="0 0 0"/>
+    <geometry>
+      <mesh filename="package://Hiwonder_description/meshes/sixth_link_1.stl" scale="0.001 0.001 0.001"/>
+    </geometry>
+  </collision>
+</link>
+<link name="fourth_link_1">
+  <inertial>
+    <origin xyz="0.029415116021796684 0.02350618639049401 2.928660555476248e-05" rpy="0 0 0"/>
+    <mass value="0.29239025387829376"/>
+    <inertia ixx="0.000208" iyy="8.1e-05" izz="0.000266" ixy="-2e-06" iyz="-0.0" ixz="0.0"/>
+  </inertial>
+  <visual>
+    <origin xyz="0.02878 -0.150304 -0.095854" rpy="0 0 0"/>
+    <geometry>
+      <mesh filename="package://Hiwonder_description/meshes/fourth_link_1.stl" scale="0.001 0.001 0.001"/>
+    </geometry>
+    <material name="silver"/>
+  </visual>
+  <collision>
+    <origin xyz="0.02878 -0.150304 -0.095854" rpy="0 0 0"/>
+    <geometry>
+      <mesh filename="package://Hiwonder_description/meshes/fourth_link_1.stl" scale="0.001 0.001 0.001"/>
+    </geometry>
+  </collision>
+</link>
+<link name="fifth_link_1">
+  <inertial>
+    <origin xyz="0.024821079126874524 0.019918646651746308 0.009994548839560524" rpy="0 0 0"/>
+    <mass value="0.293803405398946"/>
+    <inertia ixx="0.000201" iyy="0.000102" izz="0.000168" ixy="6e-06" iyz="1e-06" ixz="1e-06"/>
+  </inertial>
+  <visual>
+    <origin xyz="0.03018 -0.238894 -0.095884" rpy="0 0 0"/>
+    <geometry>
+      <mesh filename="package://Hiwonder_description/meshes/fifth_link_1.stl" scale="0.001 0.001 0.001"/>
+    </geometry>
+    <material name="silver"/>
+  </visual>
+  <collision>
+    <origin xyz="0.03018 -0.238894 -0.095884" rpy="0 0 0"/>
+    <geometry>
+      <mesh filename="package://Hiwonder_description/meshes/fifth_link_1.stl" scale="0.001 0.001 0.001"/>
+    </geometry>
+  </collision>
+</link>
 <link name="third_link_1">
   <inertial>
-    <origin xyz="-0.027698296621942956 0.04765413999012262 0.020748432672287473" rpy="0 0 0"/>
-    <mass value="0.16226233466168985"/>
-    <inertia ixx="0.000203" iyy="0.000132" izz="0.00026" ixy="-0.0" iyz="-6.9e-05" ixz="-0.0"/>
-  </inertial>
-  <visual>
-    <origin xyz="-0.028042 -0.046304 -0.095801" rpy="0 0 0"/>
+    <origin xyz="-0.027698779003945215 0.051975132993045764 2.647541288663957e-05" rpy="0 0 0"/>
+    <mass value="0.162262457476611"/>
+    <inertia ixx="0.000203" iyy="0.000102" izz="0.00029" ixy="-0.0" iyz="-0.0" ixz="0.0"/>
+  </inertial>
+  <visual>
+    <origin xyz="-0.02722 -0.046304 -0.095801" rpy="0 0 0"/>
     <geometry>
       <mesh filename="package://Hiwonder_description/meshes/third_link_1.stl" scale="0.001 0.001 0.001"/>
@@ -58,5 +118,5 @@
   </visual>
   <collision>
-    <origin xyz="-0.028042 -0.046304 -0.095801" rpy="0 0 0"/>
+    <origin xyz="-0.02722 -0.046304 -0.095801" rpy="0 0 0"/>
     <geometry>
       <mesh filename="package://Hiwonder_description/meshes/third_link_1.stl" scale="0.001 0.001 0.001"/>
@@ -64,61 +124,21 @@
   </collision>
 </link>
-<link name="fourth_link_1">
-  <inertial>
-    <origin xyz="-0.02572686990818987 0.004053928250455058 0.023157892432834615" rpy="0 0 0"/>
-    <mass value="0.2923899366437736"/>
-    <inertia ixx="0.000208" iyy="0.00026" izz="8.7e-05" ixy="-0.0" iyz="-3.2e-05" ixz="-2e-06"/>
-  </inertial>
-  <visual>
-    <origin xyz="-0.028042 -0.141658 -0.137318" rpy="0 0 0"/>
-    <geometry>
-      <mesh filename="package://Hiwonder_description/meshes/fourth_link_1.stl" scale="0.001 0.001 0.001"/>
-    </geometry>
-    <material name="silver"/>
-  </visual>
-  <collision>
-    <origin xyz="-0.028042 -0.141658 -0.137318" rpy="0 0 0"/>
-    <geometry>
-      <mesh filename="package://Hiwonder_description/meshes/fourth_link_1.stl" scale="0.001 0.001 0.001"/>
-    </geometry>
-  </collision>
-</link>
-<link name="fifth_link_1">
-  <inertial>
-    <origin xyz="0.02482151135065362 -0.01754474473381723 0.013754851957438224" rpy="0 0 0"/>
-    <mass value="0.29380221652800204"/>
-    <inertia ixx="0.000201" iyy="0.000157" izz="0.000113" ixy="-4e-06" iyz="2.4e-05" ixz="5e-06"/>
-  </inertial>
-  <visual>
-    <origin xyz="0.0285 -0.157021 -0.224566" rpy="0 0 0"/>
-    <geometry>
-      <mesh filename="package://Hiwonder_description/meshes/fifth_link_1.stl" scale="0.001 0.001 0.001"/>
-    </geometry>
-    <material name="silver"/>
-  </visual>
-  <collision>
-    <origin xyz="0.0285 -0.157021 -0.224566" rpy="0 0 0"/>
-    <geometry>
-      <mesh filename="package://Hiwonder_description/meshes/fifth_link_1.stl" scale="0.001 0.001 0.001"/>
-    </geometry>
-  </collision>
-</link>
-<link name="sixth_link_1">
-  <inertial>
-    <origin xyz="-5.564917727016649e-05 -0.024329962527568846 0.039653341169548384" rpy="0 0 0"/>
-    <mass value="0.5747761409814244"/>
-    <inertia ixx="0.000539" iyy="0.000285" izz="0.000328" ixy="-9e-06" iyz="5.9e-05" ixz="-2e-06"/>
-  </inertial>
-  <visual>
-    <origin xyz="0.003224 -0.127901 -0.28191" rpy="0 0 0"/>
-    <geometry>
-      <mesh filename="package://Hiwonder_description/meshes/sixth_link_1.stl" scale="0.001 0.001 0.001"/>
-    </geometry>
-    <material name="silver"/>
-  </visual>
-  <collision>
-    <origin xyz="0.003224 -0.127901 -0.28191" rpy="0 0 0"/>
-    <geometry>
-      <mesh filename="package://Hiwonder_description/meshes/sixth_link_1.stl" scale="0.001 0.001 0.001"/>
+<link name="left_finger_1">
+  <inertial>
+    <origin xyz="0.10077586565386246 -0.2951398577015533 -0.024100390242242975" rpy="0 0 0"/>
+    <mass value="0.016905829223014094"/>
+    <inertia ixx="7e-06" iyy="5e-06" izz="6e-06" ixy="1e-06" iyz="2e-06" ixz="-0.0"/>
+  </inertial>
+  <visual>
+    <origin xyz="0.102737 -0.696581 -0.092807" rpy="0 0 0"/>
+    <geometry>
+      <mesh filename="package://Hiwonder_description/meshes/left_finger_1.stl" scale="0.001 0.001 0.001"/>
+    </geometry>
+    <material name="silver"/>
+  </visual>
+  <collision>
+    <origin xyz="0.102737 -0.696581 -0.092807" rpy="0 0 0"/>
+    <geometry>
+      <mesh filename="package://Hiwonder_description/meshes/left_finger_1.stl" scale="0.001 0.001 0.001"/>
     </geometry>
   </collision>
@@ -126,10 +146,10 @@
 <link name="right_finger_1">
   <inertial>
-    <origin xyz="0.3334698569050242 -0.00907267411723324 -0.01453310351807563" rpy="0 0 0"/>
-    <mass value="0.07962832262347441"/>
-    <inertia ixx="4.1e-05" iyy="3.8e-05" izz="2.4e-05" ixy="3e-06" iyz="-1.2e-05" ixz="1e-05"/>
-  </inertial>
-  <visual>
-    <origin xyz="0.336601 -0.108453 -0.384364" rpy="0 0 0"/>
+    <origin xyz="0.09580963018641239 -0.2972024291150857 0.08107960390528858" rpy="0 0 0"/>
+    <mass value="0.016905829223014094"/>
+    <inertia ixx="7e-06" iyy="5e-06" izz="6e-06" ixy="-1e-06" iyz="-2e-06" ixz="-0.0"/>
+  </inertial>
+  <visual>
+    <origin xyz="0.102838 -0.697104 -0.070113" rpy="0 0 0"/>
     <geometry>
       <mesh filename="package://Hiwonder_description/meshes/right_finger_1.stl" scale="0.001 0.001 0.001"/>
@@ -138,5 +158,5 @@
   </visual>
   <collision>
-    <origin xyz="0.336601 -0.108453 -0.384364" rpy="0 0 0"/>
+    <origin xyz="0.102838 -0.697104 -0.070113" rpy="0 0 0"/>
     <geometry>
       <mesh filename="package://Hiwonder_description/meshes/right_finger_1.stl" scale="0.001 0.001 0.001"/>
@@ -144,21 +164,41 @@
   </collision>
 </link>
-<link name="left_finger_1">
-  <inertial>
-    <origin xyz="0.0021544872810023447 -0.02302381129656561 0.005335867881885781" rpy="0 0 0"/>
-    <mass value="0.07506411850762539"/>
-    <inertia ixx="3.9e-05" iyy="1.2e-05" izz="3.7e-05" ixy="-1e-06" iyz="3e-06" ixz="0.0"/>
-  </inertial>
-  <visual>
-    <origin xyz="0.014763 -0.085594 -0.345323" rpy="0 0 0"/>
-    <geometry>
-      <mesh filename="package://Hiwonder_description/meshes/left_finger_1.stl" scale="0.001 0.001 0.001"/>
-    </geometry>
-    <material name="silver"/>
-  </visual>
-  <collision>
-    <origin xyz="0.014763 -0.085594 -0.345323" rpy="0 0 0"/>
-    <geometry>
-      <mesh filename="package://Hiwonder_description/meshes/left_finger_1.stl" scale="0.001 0.001 0.001"/>
+<link name="left_silicone_1">
+  <inertial>
+    <origin xyz="4.687864967756108e-05 -0.00020343105991710297 0.0107648753930749" rpy="0 0 0"/>
+    <mass value="0.01625853008781884"/>
+    <inertia ixx="2e-06" iyy="6e-06" izz="5e-06" ixy="0.0" iyz="0.0" ixz="0.0"/>
+  </inertial>
+  <visual>
+    <origin xyz="0.005817 -0.413386 -0.064354" rpy="0 0 0"/>
+    <geometry>
+      <mesh filename="package://Hiwonder_description/meshes/left_silicone_1.stl" scale="0.001 0.001 0.001"/>
+    </geometry>
+    <material name="silver"/>
+  </visual>
+  <collision>
+    <origin xyz="0.005817 -0.413386 -0.064354" rpy="0 0 0"/>
+    <geometry>
+      <mesh filename="package://Hiwonder_description/meshes/left_silicone_1.stl" scale="0.001 0.001 0.001"/>
+    </geometry>
+  </collision>
+</link>
+<link name="right_ilicone_1">
+  <inertial>
+    <origin xyz="-4.7089655312079065e-05 0.00020383228202164316 -0.010764495822386339" rpy="0 0 0"/>
+    <mass value="0.01625853008781884"/>
+    <inertia ixx="2e-06" iyy="6e-06" izz="5e-06" ixy="0.0" iyz="0.0" ixz="0.0"/>
+  </inertial>
+  <visual>
+    <origin xyz="0.003073 -0.411641 -0.155993" rpy="0 0 0"/>
+    <geometry>
+      <mesh filename="package://Hiwonder_description/meshes/right_ilicone_1.stl" scale="0.001 0.001 0.001"/>
+    </geometry>
+    <material name="silver"/>
+  </visual>
+  <collision>
+    <origin xyz="0.003073 -0.411641 -0.155993" rpy="0 0 0"/>
+    <geometry>
+      <mesh filename="package://Hiwonder_description/meshes/right_ilicone_1.stl" scale="0.001 0.001 0.001"/>
     </geometry>
   </collision>
@@ -171,45 +211,55 @@
   <limit upper="1.570796" lower="-1.570796" effort="100" velocity="100"/>
 </joint>
-<joint name="Revolute 14" type="revolute">
-  <origin xyz="0.028042 -0.01 0.035" rpy="0 0 0"/>
-  <parent link="second_link_1"/>
-  <child link="third_link_1"/>
-  <axis xyz="-1.0 -0.0 -0.0"/>
-  <limit upper="0.785398" lower="-2.094395" effort="100" velocity="100"/>
-</joint>
-<joint name="Revolute 15" type="revolute">
-  <origin xyz="0.0 0.095354 0.041517" rpy="0 0 0"/>
+<joint name="Revolute 19" type="revolute">
+  <origin xyz="0.025276 0.064287 0.001888" rpy="0 0 0"/>
+  <parent link="fifth_link_1"/>
+  <child link="sixth_link_1"/>
+  <axis xyz="-0.004192 -0.999812 -0.018919"/>
+  <limit upper="3.141593" lower="0.0" effort="100" velocity="100"/>
+</joint>
+<joint name="Revolute 34" type="revolute">
+  <origin xyz="-0.056 0.104 5.3e-05" rpy="0 0 0"/>
   <parent link="third_link_1"/>
   <child link="fourth_link_1"/>
-  <axis xyz="-1.0 -0.0 -0.0"/>
-  <limit upper="2.879793" lower="-0.261799" effort="100" velocity="100"/>
-</joint>
-<joint name="Revolute 16" type="revolute">
-  <origin xyz="-0.056542 0.015363 0.087248" rpy="0 0 0"/>
+  <axis xyz="1.0 0.0 0.0"/>
+  <limit upper="3.141593" lower="0.0" effort="100" velocity="100"/>
+</joint>
+<joint name="Revolute 35" type="revolute">
+  <origin xyz="-0.0014 0.08859 3e-05" rpy="0 0 0"/>
   <parent link="fourth_link_1"/>
   <child link="fifth_link_1"/>
   <axis xyz="1.0 0.0 0.0"/>
-  <limit upper="0.698132" lower="-2.443461" effort="100" velocity="100"/>
-</joint>
-<joint name="Revolute 19" type="revolute">
-  <origin xyz="0.025276 -0.02912 0.057344" rpy="0 0 0"/>
-  <parent link="fifth_link_1"/>
-  <child link="sixth_link_1"/>
-  <axis xyz="-0.004192 0.443437 -0.896296"/>
+  <limit upper="1.570796" lower="0.0" effort="100" velocity="100"/>
+</joint>
+<joint name="Revolute 36" type="revolute">
+  <origin xyz="0.02722 -0.01 0.035" rpy="0 0 0"/>
+  <parent link="second_link_1"/>
+  <child link="third_link_1"/>
+  <axis xyz="1.0 0.0 0.0"/>
   <limit upper="3.141593" lower="0.0" effort="100" velocity="100"/>
 </joint>
-<joint name="Slider 29" type="prismatic">
-  <origin xyz="-0.333377 -0.019448 0.102454" rpy="0 0 0"/>
+<joint name="Slider 37" type="prismatic">
+  <origin xyz="-0.097833 0.3934 -0.004965" rpy="0 0 0"/>
+  <parent link="sixth_link_1"/>
+  <child link="left_finger_1"/>
+  <axis xyz="-0.00438 0.018937 -0.999811"/>
+  <limit upper="0.02" lower="-0.01" effort="100" velocity="100"/>
+</joint>
+<joint name="Slider 38" type="prismatic">
+  <origin xyz="-0.097934 0.393923 -0.027659" rpy="0 0 0"/>
   <parent link="sixth_link_1"/>
   <child link="right_finger_1"/>
-  <axis xyz="0.045686 0.895452 0.442806"/>
-  <limit upper="0.01" lower="-0.01" effort="100" velocity="100"/>
-</joint>
-<joint name="Slider 31" type="prismatic">
-  <origin xyz="-0.011539 -0.042307 0.063413" rpy="0 0 0"/>
-  <parent link="sixth_link_1"/>
-  <child link="left_finger_1"/>
-  <axis xyz="0.045686 0.895452 0.442806"/>
-  <limit upper="0.01" lower="-0.01" effort="100" velocity="100"/>
+  <axis xyz="-0.00438 0.018937 -0.999811"/>
+  <limit upper="0.01" lower="-0.02" effort="100" velocity="100"/>
+</joint>
+<joint name="Rigid 39" type="fixed">
+  <origin xyz="0.09692 -0.283195 -0.028453" rpy="0 0 0"/>
+  <parent link="left_finger_1"/>
+  <child link="left_silicone_1"/>
+</joint>
+<joint name="Rigid 40" type="fixed">
+  <origin xyz="0.099765 -0.285463 0.08588" rpy="0 0 0"/>
+  <parent link="right_finger_1"/>
+  <child link="right_ilicone_1"/>
 </joint>
 </robot>

File: assets/_Hiwonder_description/Hiwonder.urdf (robot description, URDF)
Before this commit: robot Hiwonder, 10 links, 9 joints
Links:
- removed link left_silicone_1
- removed link right_ilicone_1
- link fifth_link_1: mass 0.293803405398946 -> 0.29380221652800204
- link fourth_link_1: mass 0.29239025387829376 -> 0.2923899366437736
- link left_finger_1: mass 0.016905829223014094 -> 0.07506411850762539
- link right_finger_1: mass 0.016905829223014094 -> 0.07962832262347441
- link third_link_1: mass 0.162262457476611 -> 0.16226233466168985
Joints:
- removed joint Revolute 34
- removed joint Revolute 35
- removed joint Revolute 36
- removed joint Rigid 39
- removed joint Rigid 40
- removed joint Slider 37
- removed joint Slider 38
- added joint Revolute 14: type revolute, parent second_link_1, child third_link_1, origin xyz=0.028042 -0.01 0.035 rpy=-0.349066 0 0, axis 1.0 0.0 0.0, limit lower=0.0 upper=2.879793 effort=100 velocity=100
- added joint Revolute 15: type revolute, parent third_link_1, child fourth_link_1, origin xyz=0.0 0.095354 0.041517 rpy=-0.977384 0 0, axis 1.0 0.0 0.0, limit lower=0.0 upper=1.570796 effort=100 velocity=100
- added joint Revolute 16: type revolute, parent fourth_link_1, child fifth_link_1, origin xyz=-0.056542 0.015363 0.087248 rpy=-0.628319 0 0, axis 1.0 0.0 0.0, limit lower=0.0 upper=1.570796 effort=100 velocity=100
- added joint Slider 29: type prismatic, parent sixth_link_1, child right_finger_1, origin xyz=-0.333377 -0.019448 0.102454 rpy=0 0 0, axis 0.045686 0.895452 0.442806, limit lower=-0.05 upper=0.01 effort=100 velocity=100
- added joint Slider 31: type prismatic, parent sixth_link_1, child left_finger_1, origin xyz=-0.011539 -0.042307 0.063413 rpy=0 0 0, axis 0.045686 0.895452 0.442806, limit lower=-0.01 upper=0.05 effort=100 velocity=100, mimic joint=Slider 29 multiplier=-1.0 offset=0.0
- joint Revolute 13: axis 0.0 0.0 -1.0 -> 0.0 0.0 1.0; limit lower=-1.570796 upper=1.570796 effort=100 velocity=100 -> lower=0.0 upper=3.141593 effort=100 velocity=100; origin xyz=0.0 0.056304 0.060801 rpy=0 0 0 -> xyz=0.0 0.056304 0.060801 rpy=0 0 4.450589
- joint Revolute 19: axis -0.004192 -0.999812 -0.018919 -> 0.004192 -0.443437 0.896296; origin xyz=0.025276 0.064287 0.001888 rpy=0 0 0 -> xyz=0.025276 -0.02912 0.057344 rpy=-0.463617 0.455242 -1.570777
